Commit message: Fix plugins description in URDF

File: thymio_description/thymio.urdf.xacro (robot description, xacro)
@@ -6,37 +6,7 @@
     <link name="${name}_link">
       <inertial>
-        <mass value="0.0000001"/>
-        <inertia
-          ixx="1e-3" ixy="0" ixz="0"
-          iyy="1e-3" iyz="0"
-          izz="1e-3" />
+        <mass value="1e-3"/>
+        <inertia ixx="1e-3" ixy="0" ixz="0" iyy="1e-3" iyz="0" izz="1e-3"/>
       </inertial>
-      <gazebo reference="${name}_link">
-        <sensor name="${name}_sensor" type="ray">
-          <visualize>true</visualize>
-          <update_rate>${update_rate}</update_rate>
-          <always_on>true</always_on>
-          <ray>
-            <range>
-              <min>${range_min}</min>
-              <max>${range_max}</max>
-              <resolution>${resolution}</resolution>
-            </range>
-            <noise>
-              <type>gaussian</type>
-              <mean>0.0</mean>
-              <stddev>${resolution/2}</stddev>
-            </noise>
-          </ray>
-          <plugin name="${name}_controller" filename="libgazebo_ros_range.so">
-            <alwaysOn>true</alwaysOn>
-            <updateRate>${update_rate}</updateRate>
-            <robotNamespace>${robot_ns}</robotNamespace>
-            <frameName>${name}_link</frameName>
-            <topicName>${name}</topicName>
-            <radiation>infrared</radiation>
-          </plugin>
-        </sensor>
-      </gazebo>
     </link>
     <joint name="${name}_joint" type="fixed">
@@ -45,4 +15,27 @@
       <child link="${name}_link"/>
     </joint>
+    <gazebo reference="${name}_link">
+      <sensor name="${name}_sensor" type="ray">
+        <visualize>true</visualize>
+        <update_rate>${update_rate}</update_rate>
+        <always_on>true</always_on>
+        <ray>
+          <range>
+            <min>${range_min}</min>
+            <max>${range_max}</max>
+            <resolution>${resolution}</resolution>
+          </range>
+        </ray>
+        <plugin name="${name}_controller" filename="libgazebo_ros_range.so">
+          <alwaysOn>true</alwaysOn>
+          <updateRate>${update_rate}</updateRate>
+          <robotNamespace>${robot_ns}</robotNamespace>
+          <frameName>${name}_link</frameName>
+          <topicName>${name}</topicName>
+          <radiation>infrared</radiation>
+          <gaussianNoise>${resolution/2}</gaussianNoise>
+        </plugin>
+      </sensor>
+    </gazebo>
   </xacro:macro>
   <xacro:macro name="thymio_robot">
@@ -80,4 +73,9 @@
       <origin xyz="-0.025 0.047 0.013"/>
     </joint>
+    <gazebo reference="base_link">
+      <selfCollide>true</selfCollide>
+      <mu1>0.0</mu1>
+      <mu2>0.0</mu2>
+    </gazebo>
     <link name="left_wheel_link">
       <inertial>
@@ -129,4 +127,23 @@
     <xacro:proximity_sensor name="ground_left" xyz="0.04657 0.01155 0.0" rpy="0 1.5708 0"/>
     <xacro:proximity_sensor name="ground_right" xyz="0.04657 -0.01155 0.0" rpy="0 1.5708 0"/>
+    <gazebo>
+      <plugin name="differential_drive_controller" filename="libgazebo_ros_diff_drive.so">
+        <alwaysOn>true</alwaysOn>
+        <updateRate>100</updateRate>
+        <leftJoint>right_wheel_joint</leftJoint>
+        <rightJoint>left_wheel_joint</rightJoint>
+        <wheelSeparation>0.0955</wheelSeparation>
+        <wheelDiameter>0.044</wheelDiameter>
+        <torque>0.005</torque>
+        <commandTopic>cmd_vel</commandTopic>
+        <odometryTopic>odom</odometryTopic>
+        <odometryFrame>odom</odometryFrame>
+        <publishWheelJointState>true</publishWheelJointState>
+        <publishWheelTF>true</publishWheelTF>
+        <publishTf>1</publishTf>
+        <robotNamespace>${robot_ns}</robotNamespace>
+        <robotBaseFrame>base_link</robotBaseFrame>
+      </plugin>
+    </gazebo>
   </xacro:macro>
   <xacro:thymio_robot />

Commit message: Adjust proximity sensors locations and params

File: thymio_description/thymio.urdf.xacro (robot description, xacro)
@@ -3,5 +3,5 @@
   <xacro:arg name="robot_ns" default="thymio"/>
   <xacro:property name="robot_ns" value="$(arg robot_ns)"/>
-  <xacro:macro name="proximity_sensor" params="name parent_link:=base_link xyz rpy update_rate:=15 range_min:=0.01 range_max:=0.200 resolution:=0.01">
+  <xacro:macro name="proximity_sensor" params="name parent_link:=base_link xyz rpy update_rate:=10 range_min:=0.005 range_max:=0.06 resolution:=0.005 fov:=0.4">
     <link name="${name}_link">
       <inertial>
@@ -31,7 +31,8 @@
           <updateRate>${update_rate}</updateRate>
           <robotNamespace>${robot_ns}</robotNamespace>
-          <frameName>${name}_link</frameName>
+          <frameName>${robot_ns}/${name}_link</frameName>
           <topicName>${name}</topicName>
           <radiation>infrared</radiation>
+          <fov>${fov}</fov>
           <gaussianNoise>${resolution/2}</gaussianNoise>
         </plugin>
@@ -118,5 +119,5 @@
       </visual>
     </link>
-    <xacro:proximity_sensor name="proximity_center" xyz="0.055 0 0.026" rpy="0 0 0"/>
+    <!--xacro:proximity_sensor name="proximity_center" xyz="0.055 0 0.026" rpy="0 0 0"/>
     <xacro:proximity_sensor name="proximity_center_left" xyz="0.0509 0.0252 0.026" rpy="0 0 0.32"/>
     <xacro:proximity_sensor name="proximity_center_right" xyz="0.0509 -0.0252 0.026" rpy="0 0 -0.32"/>
@@ -126,5 +127,14 @@
     <xacro:proximity_sensor name="proximity_rear_right" xyz="-0.055 -0.03 0.026" rpy="0 0 3.14159"/>
     <xacro:proximity_sensor name="ground_left" xyz="0.04657 0.01155 0.0" rpy="0 1.5708 0"/>
-    <xacro:proximity_sensor name="ground_right" xyz="0.04657 -0.01155 0.0" rpy="0 1.5708 0"/>
+    <xacro:proximity_sensor name="ground_right" xyz="0.04657 -0.01155 0.0" rpy="0 1.5708 0"/-->
+    <xacro:proximity_sensor name="proximity_center" xyz="0.055 0 0.026" rpy="0 0 0"/>
+    <xacro:proximity_sensor name="proximity_center_left" xyz="0.0506 0.0261 0.026" rpy="0 0 0.33161"/>
+    <xacro:proximity_sensor name="proximity_center_right" xyz="0.0506 -0.0261 0.026" rpy="0 0 -0.33161"/>
+    <xacro:proximity_sensor name="proximity_left" xyz="0.0380 0.0493 0.026" rpy="0 0 0.66323"/>
+    <xacro:proximity_sensor name="proximity_right" xyz="0.0380 -0.0493 0.026" rpy="0 0 -0.66323"/>
+    <xacro:proximity_sensor name="proximity_rear_left" xyz="-0.055 0.0305 0.026" rpy="0 0 3.14159"/>
+    <xacro:proximity_sensor name="proximity_rear_right" xyz="-0.055 -0.0305 0.026" rpy="0 0 3.14159"/>
+    <xacro:proximity_sensor name="ground_left" xyz="0.04657 0.01155 0.0" rpy="0 1.5708 0.24311"/>
+    <xacro:proximity_sensor name="ground_right" xyz="0.04657 -0.01155 0.0" rpy="0 1.5708 -0.24311"/>
     <gazebo>
       <plugin name="differential_drive_controller" filename="libgazebo_ros_diff_drive.so">
@@ -135,5 +145,5 @@
         <wheelSeparation>0.0955</wheelSeparation>
         <wheelDiameter>0.044</wheelDiameter>
-        <torque>0.005</torque>
+        <wheelTorque>0.005</wheelTorque>
         <commandTopic>cmd_vel</commandTopic>
         <odometryTopic>odom</odometryTopic>

Commit message: Attempt to fix ROS namespacing

File: thymio_description/thymio.urdf.xacro (robot description, xacro)
@@ -1,7 +1,13 @@
 <?xml version="1.0"?>
 <robot xmlns:xacro="http://www.ros.org/wiki/xacro" name="thymio">
-  <xacro:arg name="robot_ns" default="thymio"/>
-  <xacro:property name="robot_ns" value="$(arg robot_ns)"/>
-  <xacro:macro name="proximity_sensor" params="name parent_link:=base_link xyz rpy update_rate:=10 range_min:=0.005 range_max:=0.06 resolution:=0.005 fov:=0.4">
+  <xacro:arg name="use_ns" default="0"/>
+  <xacro:arg name="robot_ns" default=""/>
+  <xacro:if value="$(arg use_ns)">
+    <xacro:property name="robot_ns" value="$(arg robot_ns)"/>
+  </xacro:if>
+  <xacro:unless value="$(arg use_ns)">
+    <xacro:property name="robot_ns" value=""/>
+  </xacro:unless>
+  <xacro:macro name="proximity_sensor" params="name topic_name parent_link:=base_link xyz rpy update_rate:=10 range_min:=0.005 range_max:=0.06 resolution:=0.005 fov:=0.4">
     <link name="${name}_link">
       <inertial>
@@ -30,7 +36,9 @@
           <alwaysOn>true</alwaysOn>
           <updateRate>${update_rate}</updateRate>
-          <robotNamespace>${robot_ns}</robotNamespace>
+          <xacro:if value="$(arg use_ns)">
+            <robotNamespace>${robot_ns}</robotNamespace>
+          </xacro:if>
           <frameName>${robot_ns}/${name}_link</frameName>
-          <topicName>${name}</topicName>
+          <topicName>${topic_name}</topicName>
           <radiation>infrared</radiation>
           <fov>${fov}</fov>
@@ -128,13 +136,13 @@
     <xacro:proximity_sensor name="ground_left" xyz="0.04657 0.01155 0.0" rpy="0 1.5708 0"/>
     <xacro:proximity_sensor name="ground_right" xyz="0.04657 -0.01155 0.0" rpy="0 1.5708 0"/-->
-    <xacro:proximity_sensor name="proximity_center" xyz="0.055 0 0.026" rpy="0 0 0"/>
-    <xacro:proximity_sensor name="proximity_center_left" xyz="0.0506 0.0261 0.026" rpy="0 0 0.33161"/>
-    <xacro:proximity_sensor name="proximity_center_right" xyz="0.0506 -0.0261 0.026" rpy="0 0 -0.33161"/>
-    <xacro:proximity_sensor name="proximity_left" xyz="0.0380 0.0493 0.026" rpy="0 0 0.66323"/>
-    <xacro:proximity_sensor name="proximity_right" xyz="0.0380 -0.0493 0.026" rpy="0 0 -0.66323"/>
-    <xacro:proximity_sensor name="proximity_rear_left" xyz="-0.055 0.0305 0.026" rpy="0 0 3.14159"/>
-    <xacro:proximity_sensor name="proximity_rear_right" xyz="-0.055 -0.0305 0.026" rpy="0 0 3.14159"/>
-    <xacro:proximity_sensor name="ground_left" xyz="0.04657 0.01155 0.0" rpy="0 1.5708 0.24311"/>
-    <xacro:proximity_sensor name="ground_right" xyz="0.04657 -0.01155 0.0" rpy="0 1.5708 -0.24311"/>
+    <xacro:proximity_sensor name="proximity_center" topic_name="proximity/center" xyz="0.055 0 0.026" rpy="0 0 0"/>
+    <xacro:proximity_sensor name="proximity_center_left" topic_name="proximity/center_left" xyz="0.0506 0.0261 0.026" rpy="0 0 0.33161"/>
+    <xacro:proximity_sensor name="proximity_center_right" topic_name="proximity/center_right" xyz="0.0506 -0.0261 0.026" rpy="0 0 -0.33161"/>
+    <xacro:proximity_sensor name="proximity_left" topic_name="proximity/left" xyz="0.0380 0.0493 0.026" rpy="0 0 0.66323"/>
+    <xacro:proximity_sensor name="proximity_right" topic_name="proximity/right" xyz="0.0380 -0.0493 0.026" rpy="0 0 -0.66323"/>
+    <xacro:proximity_sensor name="proximity_rear_left" topic_name="proximity/rear_left" xyz="-0.055 0.0305 0.026" rpy="0 0 3.14159"/>
+    <xacro:proximity_sensor name="proximity_rear_right" topic_name="proximity/rear_right" xyz="-0.055 -0.0305 0.026" rpy="0 0 3.14159"/>
+    <xacro:proximity_sensor name="ground_left" topic_name="ground/left" xyz="0.04657 0.01155 0.0" rpy="0 1.5708 0.24311"/>
+    <xacro:proximity_sensor name="ground_right" topic_name="ground/right" xyz="0.04657 -0.01155 0.0" rpy="0 1.5708 -0.24311"/>
     <gazebo>
       <plugin name="differential_drive_controller" filename="libgazebo_ros_diff_drive.so">
@@ -152,5 +160,7 @@
         <publishWheelTF>true</publishWheelTF>
         <publishTf>1</publishTf>
-        <robotNamespace>${robot_ns}</robotNamespace>
+        <xacro:if value="$(arg use_ns)">
+          <robotNamespace>${robot_ns}</robotNamespace>
+        </xacro:if>
         <robotBaseFrame>base_link</robotBaseFrame>
       </plugin>

Commit message: Fix-up: namespaces

File: thymio_description/thymio.urdf.xacro (robot description, xacro)
@@ -1,12 +1,6 @@
 <?xml version="1.0"?>
 <robot xmlns:xacro="http://www.ros.org/wiki/xacro" name="thymio">
-  <xacro:arg name="use_ns" default="0"/>
+  <xacro:arg name="use_ns" default="false"/>
   <xacro:arg name="robot_ns" default=""/>
-  <xacro:if value="$(arg use_ns)">
-    <xacro:property name="robot_ns" value="$(arg robot_ns)"/>
-  </xacro:if>
-  <xacro:unless value="$(arg use_ns)">
-    <xacro:property name="robot_ns" value=""/>
-  </xacro:unless>
   <xacro:macro name="proximity_sensor" params="name topic_name parent_link:=base_link xyz rpy update_rate:=10 range_min:=0.005 range_max:=0.06 resolution:=0.005 fov:=0.4">
     <link name="${name}_link">
@@ -37,7 +31,10 @@
           <updateRate>${update_rate}</updateRate>
           <xacro:if value="$(arg use_ns)">
-            <robotNamespace>${robot_ns}</robotNamespace>
+            <robotNamespace>$(arg robot_ns)</robotNamespace>
+            <frameName>$(arg robot_ns)/${name}_link</frameName>
           </xacro:if>
-          <frameName>${robot_ns}/${name}_link</frameName>
+          <xacro:unless value="$(arg use_ns)">
+            <frameName>${name}_link</frameName>
+          </xacro:unless>
           <topicName>${topic_name}</topicName>
           <radiation>infrared</radiation>
@@ -161,5 +158,5 @@
         <publishTf>1</publishTf>
         <xacro:if value="$(arg use_ns)">
-          <robotNamespace>${robot_ns}</robotNamespace>
+          <robotNamespace>$(arg robot_ns)</robotNamespace>
         </xacro:if>
         <robotBaseFrame>base_link</robotBaseFrame>

Commit message: Add materials

File: thymio_description/thymio.urdf.xacro (robot description, xacro)
@@ -1,4 +1,10 @@
 <?xml version="1.0"?>
 <robot xmlns:xacro="http://www.ros.org/wiki/xacro" name="thymio">
+  <material name="white">
+    <color rgba="1.0 1.0 1.0 1.0"/>
+  </material>
+  <material name="black">
+    <color rgba="0.175 0.175 0.175 1.0"/>
+  </material>
   <xacro:arg name="use_ns" default="false"/>
   <xacro:arg name="robot_ns" default=""/>
@@ -43,4 +49,5 @@
         </plugin>
       </sensor>
+      <material>Gazebo/DarkGrey</material>
     </gazebo>
   </xacro:macro>
@@ -66,11 +73,23 @@
           <mesh filename="package://thymio_description/meshes/thymio_body.dae"/>
         </geometry>
+        <material name="white"/>
       </visual>
+    </link>
+    <joint name="proximity_joint" type="fixed">
+      <parent link="base_link"/>
+      <child link="proximity"/>
+      <axis xyz="0 0 1"/>
+    </joint>
+    <link name="proximity">
       <visual>
         <geometry>
           <mesh filename="package://thymio_description/meshes/thymio_proximity_sensors.dae"/>
         </geometry>
+        <material name="black"/>
       </visual>
     </link>
+    <gazebo reference="proximity">
+      <material>Gazebo/DarkGrey</material>
+    </gazebo>
     <joint name="left_wheel_joint" type="continuous">
       <parent link="base_link"/>
@@ -83,4 +102,5 @@
       <mu1>0.0</mu1>
       <mu2>0.0</mu2>
+      <material>Gazebo/White</material>
     </gazebo>
     <link name="left_wheel_link">
@@ -99,6 +119,10 @@
           <mesh filename="package://thymio_description/meshes/thymio_left_wheel.dae"/>
         </geometry>
+        <material name="black"/>
       </visual>
     </link>
+    <gazebo reference="left_wheel_link">
+      <material>Gazebo/DarkGrey</material>
+    </gazebo>
     <joint name="right_wheel_joint" type="continuous">
       <parent link="base_link"/>
@@ -122,6 +146,10 @@
           <mesh filename="package://thymio_description/meshes/thymio_right_wheel.dae"/>
         </geometry>
+        <material name="black"/>
       </visual>
     </link>
+    <gazebo reference="right_wheel_link">
+      <material>Gazebo/DarkGrey</material>
+    </gazebo>
     <!--xacro:proximity_sensor name="proximity_center" xyz="0.055 0 0.026" rpy="0 0 0"/>
     <xacro:proximity_sensor name="proximity_center_left" xyz="0.0509 0.0252 0.026" rpy="0 0 0.32"/>
