Commit message: Add thymio_maze and cans worlds, and clean up

File: thymio_description/models/thymio.urdf.xacro (robot description, xacro)
@@ -9,5 +9,5 @@
   <xacro:arg name="use_ns" default="false"/>
   <xacro:arg name="robot_ns" default=""/>
-  <xacro:macro name="proximity_sensor" params="name topic_name parent_link:=base_link xyz rpy update_rate:=10 range_min:=0.005 range_max:=0.06 resolution:=0.005 fov:=0.4">
+  <xacro:macro name="proximity_sensor" params="name topic_name parent_link:=base_link xyz rpy update_rate:=10 range_min:=0.005 range_max:=1.0 resolution:=0.005 fov:=0.4">
     <link name="${name}_link">
       <inertial>

Commit message: Fix various paths

File: thymio_description/models/thymio.urdf.xacro (robot description, xacro)
@@ -60,5 +60,5 @@
       <collision>
         <geometry>
-          <mesh filename="package://thymio_description/meshes/thymio_body_collision.dae"/>
+          <mesh filename="package://thymio_description/models/meshes/thymio_body_collision.dae"/>
         </geometry>
       </collision>
@@ -71,5 +71,5 @@
       <visual>
         <geometry>
-          <mesh filename="package://thymio_description/meshes/thymio_body.dae"/>
+          <mesh filename="package://thymio_description/models/meshes/thymio_body.dae"/>
         </geometry>
         <material name="white"/>
@@ -84,5 +84,5 @@
       <visual>
         <geometry>
-          <mesh filename="package://thymio_description/meshes/thymio_proximity_sensors.dae"/>
+          <mesh filename="package://thymio_description/models/meshes/thymio_proximity_sensors.dae"/>
         </geometry>
         <material name="black"/>
@@ -117,5 +117,5 @@
       <visual>
         <geometry>
-          <mesh filename="package://thymio_description/meshes/thymio_left_wheel.dae"/>
+          <mesh filename="package://thymio_description/models/meshes/thymio_left_wheel.dae"/>
         </geometry>
         <material name="black"/>
@@ -144,5 +144,5 @@
       <visual>
         <geometry>
-          <mesh filename="package://thymio_description/meshes/thymio_right_wheel.dae"/>
+          <mesh filename="package://thymio_description/models/meshes/thymio_right_wheel.dae"/>
         </geometry>
         <material name="black"/>

Commit message: Add wheels friction parameters to thymio_gazebo.launch and thymio.urdf.xacro

File: thymio_description/models/thymio.urdf.xacro (robot description, xacro)
@@ -7,4 +7,8 @@
     <color rgba="0.175 0.175 0.175 1.0"/>
   </material>
+  <xacro:arg name="left_wheel_mu" default="100.0"/>
+  <xacro:property name="left_wheel_mu_p" value="$(arg left_wheel_mu)"/>
+  <xacro:arg name="right_wheel_mu" default="100.0"/>
+  <xacro:property name="right_wheel_mu_p" value="$(arg right_wheel_mu)"/>
   <xacro:arg name="use_ns" default="false"/>
   <xacro:arg name="robot_ns" default=""/>
@@ -123,4 +127,6 @@
     </link>
     <gazebo reference="left_wheel_link">
+      <mu1>${left_wheel_mu_p}</mu1>
+      <mu2>${left_wheel_mu_p / 2.0}</mu2>
       <material>Gazebo/DarkGrey</material>
     </gazebo>
@@ -150,4 +156,6 @@
     </link>
     <gazebo reference="right_wheel_link">
+      <mu1>${right_wheel_mu_p}</mu1>
+      <mu2>${right_wheel_mu_p / 2.0}</mu2>
       <material>Gazebo/DarkGrey</material>
     </gazebo>

Commit message: Parametrize Thymio mass
80% of mass is assigned to the body and 10% to each wheel.

File: thymio_description/models/thymio.urdf.xacro (robot description, xacro)
@@ -11,4 +11,10 @@
   <xacro:arg name="right_wheel_mu" default="100.0"/>
   <xacro:property name="right_wheel_mu_p" value="$(arg right_wheel_mu)"/>
+  <xacro:arg name="mass" default="0.200"/>
+  <xacro:property name="mass_p" value="$(arg mass)"/>
+  <!-- Body mass is 80% of total mass -->
+  <xacro:property name="body_mass" value="${mass_p * 0.80}"/>
+  <!-- Each wheel is 10% of total mass -->
+  <xacro:property name="wheel_mass" value="${mass_p * 0.10}"/>
   <xacro:arg name="use_ns" default="false"/>
   <xacro:arg name="robot_ns" default=""/>
@@ -59,6 +65,6 @@
     <link name="base_link">
       <inertial>
-        <mass value="0.200"/>
-        <inertia ixx="0.00024282" ixy="0" ixz="0" iyy="0.00023542" iyz="0" izz="0.00041073"/>
+        <mass value="${body_mass}"/>
+        <inertia ixx="${0.0012141 * body_mass}" ixy="0" ixz="0" iyy="${0.0011771 * body_mass}" iyz="0" izz="${0.00205365 * body_mass}"/>
       </inertial>
       <collision>
@@ -110,6 +116,6 @@
     <link name="left_wheel_link">
       <inertial>
-        <mass value="0.025"/>
-        <inertia ixx="0.00000363" ixy="0" ixz="0" iyy="0.00000605" iyz="0" izz="0.00000363"/>
+        <mass value="${wheel_mass}"/>
+        <inertia ixx="${0.0001452 * wheel_mass}" ixy="0" ixz="0" iyy="${0.000242 * wheel_mass}" iyz="0" izz="${0.0001452 * wheel_mass}"/>
       </inertial>
       <collision>
@@ -139,6 +145,6 @@
     <link name="right_wheel_link">
       <inertial>
-        <mass value="0.025"/>
-        <inertia ixx="0.00000363" ixy="0" ixz="0" iyy="0.00000605" iyz="0" izz="0.00000363"/>
+        <mass value="${wheel_mass}"/>
+        <inertia ixx="${0.0001452 * wheel_mass}" ixy="0" ixz="0" iyy="${0.000242 * wheel_mass}" iyz="0" izz="${0.0001452 * wheel_mass}"/>
       </inertial>
       <collision>
